File: hardware/rev-b/keychain-rev-b.kicad_sch (KiCad schematic)
At the start: 56 parts, among them J1 USB-C, J2 OLED 0.96" I2C, J3 SWD, M1 вибромотор 0820, Q1 AO3401A, Q2 AO3401A, Q3 AO3400A, Q4 AO3400A, SW1 B3U-3100P, U1 MDBT50Q-1MV2, U2 MCP73832-2, U3 USBLC6-2SC6, U4 LIS3DH, U5 LTR-303ALS-01, U6 SPH0641LM4H-1

Commit message: Плата rev B: исправления перед заказом, разведена заново
- «100k» в BOM был с номером LCSC C25086 — это не 100 кОм (у LCSC/JLCPCB
  1 Ом): на R6 закоротило бы VBUS, на R7/R9/R15 не работали бы экран и вибро.
  Теперь C25741 (0402WGF1003TCE, базовая).
- R6 10 кОм: после отключения USB Q1 открывается за ~15 мс, а не ~130 мс
  (VSYS падал до 2.5 В), утечка горячего Шоттки не поднимает VBUS.
- C11 между затвором и стоком Q2: бросок тока экрана ~0.14 А вместо
  0.6–1.3 А, VSYS не ниже 3.64 В (SPICE).
- R20 100 кОм с CHG_IO на землю: «1» статуса заряда 2.8–3.4 В вместо 3.8 В
  (выше VDD + 0.3 В).
- Ячейка на 1.4 мм ниже: не налезает на штыревой разъём экрана.
- README: модуль экрана с LDO, повороты деталей оборота в предпросмотре
  JLCPCB, зазоры ячейки и USB-C, итог проверки.

DRC: 0 ошибок, 0 несоединённых (предупреждение шелкографии — прежнее);
схема сверена с netlist.py, расхождений 0.

Co-Authored-By: Claude Opus 5.5 <noreply@anthropic.com>
Claude-Session: https://claude.ai/code/session_01RQ7GfaTDyVK1Dcdo3sKM8F
Parts:
- added R20: 100k, Resistor_SMD:R_0402_1005Metric, symbol Device:R_Small
- R15, R7, R9: LCSC C25086 -> C25741; MPN 0402WGF100KTCE -> 0402WGF1003TCE
- R6: value 100k -> 10k; LCSC C25086 -> C25744; MPN 0402WGF100KTCE -> 0402WGF1002TCE
Connections:
- net CHG_IO: now also R20.1
- net DISP_VCC: now also C11.2
- net GND: now also R20.2
- net VSYS: no longer C11.2

Commit message: Черновик: плата rev B — итоговая трассировка (TVS D3, CHG_EN P0.24, 47k, C6 4.7 мкФ), выходные файлы заново (в работе)
Co-Authored-By: Claude Opus 5.5 <noreply@anthropic.com>
Claude-Session: https://claude.ai/code/session_01RQ7GfaTDyVK1Dcdo3sKM8F
Parts:
- added D3: SMF5.0A, Diode_SMD:D_SOD-123F, symbol Device:D_Zener
- C14, C15: value 1uF -> 100nF; LCSC C52923 -> C1525; MPN CL05A105KA5NQNC -> CL05B104KO5NNNC
- C6: value 10uF -> 4.7uF; LCSC C19702 -> C19666; MPN CL10A106KP8NNNC -> CL10A475KO8NNNC
- R20: value 100k -> 47k; LCSC C25741 -> C25792; MPN 0402WGF1003TCE -> 0402WGF4702TCE
Connections:
- net GND: now also D3.2 (A); no longer R3.2, U4.7 (SDO/SA0)
- net VBUS: now also D3.1 (K)
- net VDD: now also U4.7 (SDO/SA0)
- net CHG_EN: now reaches U1.48 (P0.24)
- net CHG_EN: now also R3.2
- no-connect marks 43 -> 42
