File: hardware/rev-b/out/panel/keychain-rev-b-panel.kicad_pcb (KiCad board)
At the start: 4 copper layers, 76 x 72 mm, 162 parts, among them J1_1 USB-C, J1_2 USB-C, J2_1 OLED 0.96" I2C, J2_2 OLED 0.96" I2C, J3_1 SWD, J3_2 SWD, M1_1 вибромотор 0820, M1_2 вибромотор 0820, Q1_1 AO3401A, Q1_2 AO3401A, Q2_1 AO3401A, Q2_2 AO3401A, Q3_1 AO3400A, Q3_2 AO3400A, Q4_1 AO3400A, Q4_2 AO3400A, SW1_1 B3U-3100P, SW1_2 B3U-3100P, U1_1 MDBT50Q-1MV2, U1_2 MDBT50Q-1MV2, U2_1 MCP73832-2, U2_2 MCP73832-2, U3_1 USBLC6-2SC6, U3_2 USBLC6-2SC6, U4_1 LIS3DH, U4_2 LIS3DH, U5_1 LTR-303ALS-01, U5_2 LTR-303ALS-01, U6_1 SPH0641LM4H-1, U6_2 SPH0641LM4H-1

Commit message: Плата: метка JLCJLCJLCJLC под ячейкой, третья перемычка панели, защита генераторов, поправки поворотов как подсказка
- Номер заказа JLCPCB ляжет на метку под ячейкой (опция «Order Number (Specify Position)»),
  а не на видимый через прозрачный корпус оборот.
- Панель: каждая плата держится ещё и короткой перемычкой на нижнем крае между USB-C и
  правым винтом; вырезы заливок у перемычек, проверка меди после перезаливки.
- build.py: route и finish не трогают разведённую плату без --force, сохраняют только
  после чистого DRC, неудачный DRC — в out/work; panel не удаляет out/panel до проверки.
- fab.py: поправки поворотов U2 и J1 — лучшие догадки, их сверяют в предпросмотре JLCPCB;
  таблица точных поправок по номеру LCSC — для заполнения после первого заказа.

Co-Authored-By: Claude Opus 5.5 <noreply@anthropic.com>
Claude-Session: https://claude.ai/code/session_01RQ7GfaTDyVK1Dcdo3sKM8F
Parts:
- removed KiKit_MB_5_5, KiKit_MB_5_6, KiKit_MB_8_5: NPTH, NPTH
- added KiKit_MB_10_2: NPTH, NPTH, F.Cu at (44.5, 9.50)
- added KiKit_MB_10_3: NPTH, NPTH, F.Cu at (45.5, 9.50)
- added KiKit_MB_10_4: NPTH, NPTH, F.Cu at (46.5, 9.50)
- added KiKit_MB_7_5: NPTH, NPTH, F.Cu at (69.2, 29.7)
- added KiKit_MB_7_6: NPTH, NPTH, F.Cu at (69.2, 30.7)
- added KiKit_MB_9_2: NPTH, NPTH, F.Cu at (66.0, 56.0)
- added KiKit_MB_9_3: NPTH, NPTH, F.Cu at (65.0, 56.0)
- added KiKit_MB_9_4: NPTH, NPTH, F.Cu at (64.0, 56.0)
- added KiKit_MB_9_5: NPTH, NPTH, F.Cu at (63.0, 56.0)
- moved KiKit_MB_5_4 41.7 mm to (29.5, 62.5)
- moved KiKit_MB_5_3 41.0 mm to (30.5, 62.5)
- moved KiKit_MB_5_2 40.4 mm to (31.5, 62.5)
- moved KiKit_MB_8_2 38.1 mm to (69.2, 18.1)
- moved KiKit_MB_8_3 37.2 mm to (69.2, 19.1)
- moved KiKit_MB_8_4 36.3 mm to (69.2, 20.1)
- moved KiKit_MB_6_2 21.2 mm to (69.2, 48.0)
- moved KiKit_MB_6_3 21.2 mm to (69.2, 49.0)
- moved KiKit_MB_6_4 21.2 mm to (69.2, 50.0)
- moved KiKit_MB_6_5 21.2 mm to (69.2, 51.0)
- moved KiKit_MB_6_6 21.2 mm to (69.2, 52.0)
- moved KiKit_MB_7_2 8.67 mm to (69.2, 26.7)
- moved KiKit_MB_7_3 8.67 mm to (69.2, 27.7)
- moved KiKit_MB_7_4 8.67 mm to (69.2, 28.7)
Other:
- outline, holes or cut-outs redrawn
- board text added: "JLCJLCJLCJLC"
